File: oven-tempsensor-esp32c6.kicad_sch (KiCad schematic)
At the start: 0 parts

Commit message: First routed version - not sent to production yet
- 4-layer board
- all elements placed and routed
Parts:
- added J1: Battery, Connector_PinHeader_2.54mm:PinHeader_1x02_P2.54mm_Horizontal, symbol Connector:Conn_01x02_Pin
- added R1, R2: 100k, Resistor_SMD:R_0603_1608Metric_Pad0.98x0.95mm_HandSolder, symbol Device:R
- added R10, R11: 10k, Resistor_SMD:R_0603_1608Metric_Pad0.98x0.95mm_HandSolder, symbol Device:R
- added U1: XIAO-ESP32-C6-SMD, Chof747_MCUs:XIAO-ESP32-C6-DIP, symbol Chof747_MCUs:XIAO-ESP32-C6-SMD
Connections:
- new net +3V3: R10.1, R11.1, U1.12 (3V3_OUT), U1.22 (3V3_OUT)
- new net BAT+: J1.2 (Pin_2), R1.1, U1.23 (BAT+)
- new net BAT-: J1.1 (Pin_1), R2.1, U1.24 (BAT-)
- new net BAT_SENSE: R1.2, R2.2, U1.2 (D1)
- new net D10_ADC1DRV: U1.11 (D10)
- new net D4_SDA: R11.2, U1.5 (D4)
- new net D5_SCL: R10.2, U1.6 (D5)
- new net D7_MOD: U1.8 (D7)
- new net D8_SCD: U1.9 (D8)
- new net D9_ADC0DRV: U1.10 (D9)
- new net EN_RESET: U1.17 (EN)
- new net GND: U1.13 (GND), U1.18 (GND)
- no-connect marks 0 -> 10
Other:
- added sheet Peripherals (peripherals.kicad_sch)
- added sheet Sensing (sensing.kicad_sch)
