File: oven-tempsensor-esp32c6.kicad_pcb (KiCad board)
At the start: 2 copper layers, 2 parts

Commit message: First routed version - not sent to production yet
- 4-layer board
- all elements placed and routed
Parts:
- added C1: C, Capacitor_SMD:C_0603_1608Metric_Pad1.08x0.95mm_HandSolder, F.Cu at (187.5, 116.0)
- added C2: 0.1uF, Capacitor_SMD:C_0603_1608Metric_Pad1.08x0.95mm_HandSolder, F.Cu at (193.4, 111.0)
- added J1: Battery, Connector_PinHeader_2.54mm:PinHeader_1x02_P2.54mm_Horizontal, B.Cu at (166.0, 105.0)
- added J2: Temp 1, Chof747_Footprints:MJ2509N, B.Cu at (167.7, 85.9)
- added J3: Temp 2, Chof747_Footprints:MJ2509N, B.Cu at (153.2, 85.9)
- added J4: OLED Display, Chof747_Footprints:OLED-TH_L38.0-W12.0_HS91L02W2C01, F.Cu at (160.5, 100.3)
- added R1: 100k, Resistor_SMD:R_0603_1608Metric_Pad0.98x0.95mm_HandSolder, F.Cu at (176.8, 98.1)
- added R10: 10k, Resistor_SMD:R_0603_1608Metric_Pad0.98x0.95mm_HandSolder, F.Cu at (181.5, 87.4)
- added R11: 10k, Resistor_SMD:R_0603_1608Metric_Pad0.98x0.95mm_HandSolder, F.Cu at (184.8, 87.4)
- added R2: 100k, Resistor_SMD:R_0603_1608Metric_Pad0.98x0.95mm_HandSolder, F.Cu at (176.8, 102.6)
- added R3: 10k, Resistor_SMD:R_0603_1608Metric_Pad0.98x0.95mm_HandSolder, F.Cu at (170.5, 113.5)
- added R4: 10k, Resistor_SMD:R_0603_1608Metric_Pad0.98x0.95mm_HandSolder, F.Cu at (197.1, 111.0)
- added R5: 10k, Resistor_SMD:R_0603_1608Metric_Pad0.98x0.95mm_HandSolder, F.Cu at (185.5, 113.5)
- added R6: 2k, Resistor_SMD:R_0603_1608Metric_Pad0.98x0.95mm_HandSolder, F.Cu at (167.0, 92.4)
- added R7: 2k, Resistor_SMD:R_0603_1608Metric_Pad0.98x0.95mm_HandSolder, F.Cu at (148.9, 89.8)
- added REF**: MountingHole_3.2mm_M3, MountingHole:MountingHole_3.2mm_M3, F.Cu at (196.0, 83.7)
- added REF**: MountingHole_3.2mm_M3, MountingHole:MountingHole_3.2mm_M3, F.Cu at (150.7, 117.9)
- added SW1: Mode, Button_Switch_THT:SW_PUSH_6mm, F.Cu at (160.5, 113.5)
- added SW2: Secondary, Button_Switch_THT:SW_PUSH_6mm, F.Cu at (175.5, 113.5)
- added SW3: Reset, Button_Switch_THT:SW_PUSH_6mm, F.Cu at (190.0, 113.5)
- added U1: XIAO-ESP32-C6-SMD, Chof747_MCUs:XIAO-ESP32-C6-DIP, F.Cu at (189.4, 100.0)
- added U2: ADS1115IDGS, Package_SO:TSSOP-10_3x3mm_P0.5mm, F.Cu at (152.3, 99.2)
Routing:
- net +3V3: track 0.00 -> 127.0 mm, vias 0 -> 7
- net /D10_ADC1DRV: track 0.00 -> 62.5 mm, vias 0 -> 2
- net /D4_SDA: track 0.00 -> 62.1 mm
- net /D5_SCL: track 0.00 -> 46.6 mm, vias 0 -> 4
- net BAT+: track 0.00 -> 35.9 mm, vias 0 -> 1
- net /BAT_SENSE: track 0.00 -> 31.8 mm
- net /D9_ADC0DRV: track 0.00 -> 31.2 mm
- net BAT-: track 0.00 -> 29.8 mm, vias 0 -> 1
- net /EN_RESET: track 0.00 -> 24.4 mm
- net /D7_MOD: track 0.00 -> 23.4 mm
- net /Sensing/TEMP0: track 0.00 -> 21.5 mm, vias 0 -> 1
- net GND: track 0.00 -> 15.2 mm, vias 0 -> 10
- net /D8_SCD: track 0.00 -> 14.2 mm
- net /Sensing/TEMP1: track 0.00 -> 12.4 mm
- added copper zone on B.Cu, net GND
- added copper zone on F.Cu, net GND
- added copper zone on In1.Cu, net GND
- added copper zone on In2.Cu, net GND
Other:
- board outline added: 53 x 41.5 mm
- copper layers 2 -> 4

Commit message: Added text and fabrication
Parts:
- removed the G*** at (22.4, 182.3)
- moved G*** 187.4 mm to (187.9, 83.2), turned to 90 degrees
Other:
- board text added: "+"
- board text added: "-"
- board text added: "2"
- board text added: "Oven Temp Sensor V1.0 (c) chof 2026"
- board text added: "Temp 1"
